File: Phaser.kicad_pcb (KiCad board)
At the start: 2 copper layers, 138 x 83.3 mm, 136 parts, among them J1 9V, J10 DA3, J11 BC1, J12 DRY, J13 BC2, J14 BC3, J15 GND, J16 DC1, J17 DC2, J18 DC3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

Commit message: Cleaned up Silks
Other:
- rule pad_to_mask_clearance: 0.051 -> 0
